File: DaughterBoard/MiniRectangleDB/MiniRectangleDB.kicad_sch (KiCad schematic)
At the start: 9 parts, among them J1 USB C Connector, J4 Conn_01x06, U2 USBLC6-2SC6

Commit message: Finished main PCB
Parts:
- added U2: USBLC6-2SC6, Package_TO_SOT_SMD:SOT-23-6, symbol Power_Protection:USBLC6-2SC6
Connections:
- net 3vCable: now also U2.5 (VBUS)
- net DATA: now also U2.6 (I/O1); no longer J1.B11 (RX1+)
- net GND: now also U2.2 (GND)
- new net DATABUS: J1.B11 (RX1+), U2.1 (I/O1)
Other:
- moved on the sheet: J4
Changed lines of the file:
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@@
     )
   )
-  (global_label "DATA" (shape input) (at 108.966 84.963 180) (fields_autoplaced)
-    (effects (font (size 1.27 1.27)) (justify right))
-    (property "Intersheetrefs" "${INTERSHEET_REFS}" (at 101.6454 84.963 0)
-      (effects (font (size 1.27 1.27)) (justify right) hide)
-    )
-  )
-  (global_label "D-" (shape input) (at 108.966 77.343 180) (fields_autoplaced)
-    (effects (font (size 1.27 1.27)) (justify right))
-    (property "Intersheetrefs" "${INTERSHEET_REFS}" (at 103.2178 77.343 0)
+  (global_label "DATA" (shape input) (at 142.113 53.086 180) (fields_autoplaced)
+    (effects (font (size 1.27 1.27)) (justify right))
+    (property "Intersheetrefs" "${INTERSHEET_REFS}" (at 134.7924 53.086 0)
+      (effects (font (size 1.27 1.27)) (justify right) hide)
+    )
+  )
+  (global_label "DATA" (shape input) (at 89.281 91.313 180) (fields_autoplaced)
+    (effects (font (size 1.27 1.27)) (justify right))
+    (property "Intersheetrefs" "${INTERSHEET_REFS}" (at 81.9604 91.313 0)
+      (effects (font (size 1.27 1.27)) (justify right) hide)
+    )
+  )
+  (global_label "D-" (shape input) (at 142.113 45.466 180) (fields_autoplaced)
+    (effects (font (size 1.27 1.27)) (justify right))
+    (property "Intersheetrefs" "${INTERSHEET_REFS}" (at 136.3648 45.466 0)
       (effects (font (size 1.27 1.27)) (justify right) hide)
     )
@@
     )
   )
-  (global_label "3vCable" (shape input) (at 108.966 82.423 180) (fields_autoplaced)
-    (effects (font (size 1.27 1.27)) (justify right))
-    (property "Intersheetrefs" "${INTERSHEET_REFS}" (at 98.5613 82.423 0)
+  (global_label "3vCable" (shape input) (at 99.441 83.693 90) (fields_autoplaced)
+    (effects (font (size 1.27 1.27)) (justify left))
+    (property "Intersheetrefs" "${INTERSHEET_REFS}" (at 99.441 73.2883 90)
+      (effects (font (size 1.27 1.27)) (justify left) hide)
+    )
+  )
+  (global_label "3vCable" (shape input) (at 142.113 50.546 180) (fields_autoplaced)
+    (effects (font (size 1.27 1.27)) (justify right))
+    (property "Intersheetrefs" "${INTERSHEET_REFS}" (at 131.7083 50.546 0)
       (effects (font (size 1.27 1.27)) (justify right) hide)
     )
@@
     )
   )
-  (global_label "DATA" (shape input) (at 67.31 53.213 270) (fields_autoplaced)
-    (effects (font (size 1.27 1.27)) (justify right))
-    (property "Intersheetrefs" "${INTERSHEET_REFS}" (at 67.3894 60.0409 90)
+  (global_label "DATABUS" (shape input) (at 67.31 53.213 270) (fields_autoplaced)
+    (effects (font (size 1.27 1.27)) (justify right))
+    (property "Intersheetrefs" "${INTERSHEET_REFS}" (at 67.31 64.3436 90)
       (effects (font (size 1.27 1.27)) (justify right) hide)
     )
@@
     )
   )
-  (global_label "D+" (shape input) (at 108.966 74.803 180) (fields_autoplaced)
-    (effects (font (size 1.27 1.27)) (justify right))
-    (property "Intersheetrefs" "${INTERSHEET_REFS}" (at 103.2178 74.803 0)
+  (global_label "DATABUS" (shape input) (at 89.281 96.393 180) (fields_autoplaced)
+    (effects (font (size 1.27 1.27)) (justify right))
+    (property "Intersheetrefs" "${INTERSHEET_REFS}" (at 78.1504 96.393 0)
+      (effects (font (size 1.27 1.27)) (justify right) hide)
+    )
+  )
+  (global_label "D+" (shape input) (at 142.113 42.926 180) (fields_autoplaced)
+    (effects (font (size 1.27 1.27)) (justify right))
+    (property "Intersheetrefs" "${INTERSHEET_REFS}" (at 136.3648 42.926 0)
       (effects (font (size 1.27 1.27)) (justify right) hide)
     )
@@
     )
   )
-  (symbol (lib_id "power:+5V") (at 108.966 79.883 90) (unit 1)
-    (in_bom yes) (on_board yes) (dnp no)
-    (property "Reference" "#PWR03" (at 112.776 79.883 0)
-      (effects (font (size 1.27 1.27)) hide)
-    )
-    (property "Value" "+5V" (at 105.41 79.883 90)
-      (effects (font (size 1.27 1.27)) (justify left))
-    )
-    (property "Footprint" "" (at 108.966 79.883 0)
-      (effects (font (size 1.27 1.27)) hide)
-    )
-    (property "Datasheet" "" (at 108.966 79.883 0)
+  (symbol (lib_id "power:+5V") (at 142.113 48.006 90) (unit 1)
+    (in_bom yes) (on_board yes) (dnp no)
+    (property "Reference" "#PWR03" (at 145.923 48.006 0)
+      (effects (font (size 1.27 1.27)) hide)
+    )
+    (property "Value" "+5V" (at 138.557 48.006 90)
+      (effects (font (size 1.27 1.27)) (justify left))
+    )
+    (property "Footprint" "" (at 142.113 48.006 0)
+      (effects (font (size 1.27 1.27)) hide)
+    )
+    (property "Datasheet" "" (at 142.113 48.006 0)
       (effects (font (size 1.27 1.27)) hide)
     )
@@
     )
   )
-  (symbol (lib_name "GND_1") (lib_id "power:GND") (at 108.966 72.263 270) (unit 1)
-    (in_bom yes) (on_board yes) (dnp no)
-    (property "Reference" "#PWR052" (at 102.616 72.263 0)
-      (effects (font (size 1.27 1.27)) hide)
-    )
-    (property "Value" "GND" (at 105.791 72.263 90)
+  (symbol (lib_id "Power_Protection:USBLC6-2SC6") (at 99.441 93.853 0) (unit 1)
+    (in_bom yes) (on_board yes) (dnp no) (fields_autoplaced)
+    (property "Reference" "U2" (at 102.2097 80.5942 0)
+      (effects (font (size 1.27 1.27)) (justify left))
+    )
+    (property "Value" "USBLC6-2SC6" (at 102.2097 83.1342 0)
+      (effects (font (size 1.27 1.27)) (justify left))
+    )
+    (property "Footprint" "Package_TO_SOT_SMD:SOT-23-6" (at 99.441 106.553 0)
+      (effects (font (size 1.27 1.27)) hide)
+    )
+    (property "Datasheet" "https://www.st.com/resource/en/datasheet/usblc6-2.pdf" (at 104.521 84.963 0)
+      (effects (font (size 1.27 1.27)) hide)
+    )
+    (pin "1")
+    (pin "2")
+    (pin "3")
+    (pin "4")
+    (pin "5")
+    (pin "6")
+    (instances
+      (project "OpenRectangle"
+        (path "/0ee7bd02-e26d-4978-ae8c-675a718c78c0"
+          (reference "U2") (unit 1)
+        )
+      )
+      (project "OpenMiniRectangle"
+        (path "/798975c2-d104-4b51-bc9d-eb81d8f1bd39"
+          (reference "U2") (unit 1)
+        )
+      )
+      (project "MiniRectangleDB"
+        (path "/9b225c0b-91fc-44a4-b73d-e36704cd827b"
+          (reference "U2") (unit 1)
+        )
+      )
+    )
+  )
+  (symbol (lib_name "GND_1") (lib_id "power:GND") (at 142.113 40.386 270) (unit 1)
+    (in_bom yes) (on_board yes) (dnp no)
+    (property "Reference" "#PWR052" (at 135.763 40.386 0)
+      (effects (font (size 1.27 1.27)) hide)
+    )
+    (property "Value" "GND" (at 138.938 40.386 90)
       (effects (font (size 1.27 1.27)) (justify right))
     )
-    (property "Footprint" "" (at 108.966 72.263 0)
-      (effects (font (size 1.27 1.27)) hide)
-    )
-    (property "Datasheet" "" (at 108.966 72.263 0)
+    (property "Footprint" "" (at 142.113 40.386 0)
+      (effects (font (size 1.27 1.27)) hide)
+    )
+    (property "Datasheet" "" (at 142.113 40.386 0)
       (effects (font (size 1.27 1.27)) hide)
     )
@@
         (path "/9b225c0b-91fc-44a4-b73d-e36704cd827b"
           (reference "R1") (unit 1)
+        )
+      )
+    )
+  )
+  (symbol (lib_id "power:GND") (at 99.441 104.013 0) (unit 1)
+    (in_bom yes) (on_board yes) (dnp no) (fields_autoplaced)
+    (property "Reference" "#PWR08" (at 99.441 110.363 0)
+      (effects (font (size 1.27 1.27)) hide)
+    )
+    (property "Value" "GND" (at 99.441 108.5755 0)
+      (effects (font (size 1.27 1.27)))
+    )
+    (property "Footprint" "" (at 99.441 104.013 0)
+      (effects (font (size 1.27 1.27)) hide)
+    )
+    (property "Datasheet" "" (at 99.441 104.013 0)
+      (effects (font (size 1.27 1.27)) hide)
+    )
+    (pin "1")
+    (instances
+      (project "OpenRectangle"
+        (path "/0ee7bd02-e26d-4978-ae8c-675a718c78c0"
+          (reference "#PWR08") (unit 1)
+        )
+      )
+      (project "OpenMiniRectangle"
+        (path "/798975c2-d104-4b51-bc9d-eb81d8f1bd39"
+          (reference "#PWR013") (unit 1)
+        )
+      )
+      (project "MiniRectangleDB"
+        (path "/9b225c0b-91fc-44a4-b73d-e36704cd827b"
+          (reference "#PWR09") (unit 1)
         )
       )
@@
     )
   )
-  (symbol (lib_id "Connector_Generic:Conn_01x06") (at 114.046 77.343 0) (unit 1)
-    (in_bom yes) (on_board yes) (dnp no) (fields_autoplaced)
-    (property "Reference" "J4" (at 116.332 77.978 0)
-      (effects (font (size 1.27 1.27)) (justify left))
-    )
-    (property "Value" "Conn_01x06" (at 116.332 80.518 0)
-      (effects (font (size 1.27 1.27)) (justify left))
-    )
-    (property "Footprint" "Connector_PinHeader_2.54mm:PinHeader_1x06_P2.54mm_Vertical" (at 114.046 77.343 0)
-      (effects (font (size 1.27 1.27)) hide)
-    )
-    (property "Datasheet" "~" (at 114.046 77.343 0)
-      (effects (font (size 1.27 1.27)) hide)
-    )
+  (symbol (lib_id "Connector_Generic:Conn_01x06") (at 147.193 45.466 0) (unit 1)
+    (in_bom yes) (on_board yes) (dnp no) (fields_autoplaced)
+    (property "Reference" "J4" (at 149.479 46.101 0)
+      (effects (font (size 1.27 1.27)) (justify left))
+    )
+    (property "Value" "Conn_01x06" (at 149.479 48.641 0)
+      (effects (font (size 1.27 1.27)) (justify left))
+    )
+    (property "Footprint" "Connector_PinHeader_2.54mm:PinHeader_1x06_P2.54mm_Vertical" (at 147.193 45.466 0)
+      (effects (font (size 1.27 1.27)) hide)
+    )
+    (property "Datasheet" "~" (at 147.193 45.466 0)
+      (effects (font (size 1.27 1.27)) hide)
+    )
