File: PCB/OpenMiniRectangle.kicad_sch (KiCad schematic)
At the start: 50 parts, among them J1 USB C Connector, J2 JTAG_TC2030, J3 Conn_01x06, J4 Conn_01x06, SW1 Boot, U1 XC6206, U2 USBLC6-2SC6, U3 RP2040, U4 W25Q128JVS, Y1 12MHz

Commit message: Added separated board for the DB
Connections:
- net LED3: now reaches U3.34 (GPIO22)
- net LED2: now reaches U3.35 (GPIO23)
- net LED1: now reaches U3.36 (GPIO24)
- net HOME: now reaches U3.38 (GPIO26/ADC0)
- net PICO_LED renamed SELECT
- no-connect marks 8 -> 7
Other:
- moved on the sheet: H1, H10, H2, H3, H4, H5, H6, H7, H8, H9

Commit message: Finished main PCB
Parts:
- removed F1: 500 mA, Fuse:Fuse_1206_3216Metric, symbol Device:Fuse_Small
- removed H1: MountingHole, MountingHole:MountingHole_2.2mm_M2, symbol Mechanical:MountingHole
- removed H3: MountingHole_Pad, MountingHole:MountingHole_2.2mm_M2_DIN965_Pad, symbol Mechanical:MountingHole_Pad
- removed J1: USB C Connector, footprints:TYPE-C_24P_QCHT, symbol Connector:USB_C_Receptacle
- removed J4: Conn_01x06, Connector_PinHeader_2.54mm:PinHeader_1x06_P2.54mm_Vertical, symbol Connector_Generic:Conn_01x06
- removed R1: 1M, Resistor_SMD:R_0603_1608Metric, symbol Device:R_Small
- removed R2, R3: 5.1k, Resistor_SMD:R_0402_1005Metric, symbol Device:R_Small
- removed U2: USBLC6-2SC6, Package_TO_SOT_SMD:SOT-23-6, symbol Power_Protection:USBLC6-2SC6
- added D3, D4, D5: LED, LED_THT:LED_D3.0mm, symbol Device:LED
- added R8 (x3): 1k, Resistor_SMD:R_0603_1608Metric, symbol Device:R_Small
- renumbered H2 to H1, H6 to H2, H5 to H3, H9 to H4, H10 to H5, H7 to H6, H8 to H7, H4 to H8, J3 to J2
Connections:
- net GND: now also D3.1 (K), D4.1 (K), D5.1 (K)
- net LED1: now also R8.1
- net LED2: now also R8.1
- net LED3: now also R8.1
- new net: D5.2 (A), R8.2
- new net: D4.2 (A), R8.2
- new net: D3.2 (A), R8.2
- no-connect marks 7 -> 2
Other:
- note added: "Daughterboard"
- note added: "Indicator LEDs"
- note added: "Mounting Holes"
- note removed: "ESD Protection"
- note removed: "USB PORT"
- moved on the sheet: C1, C2, D1, D2, H1, H2, H3, H4, H5, H6, H7, H8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
